File: PiezoAMP/Piezo_Amplifier/Piezo_Amplifier.kicad_pcb (KiCad board)
At the start: 2 copper layers, 42.5 x 40.7 mm, 20 parts, among them SW1 SPST, U1 NE5534

Commit message: Cleanup
Other:
- board text added: "Piezo Mic Amplifier v1.0 Dan Larsson 2024"
- board text added: "WayWayWay"
- board text removed: "Piezo Mic Amplifier Dan Larsson 2024"
Changed lines of the file:
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@@
   (gr_line (start 58.75 42.75) (end 97.3 42.75)
     (stroke (width 0.1) (type default)) (layer "Edge.Cuts"))
-  (gr_text "Piezo Mic Amplifier\nDan Larsson 2024" (at 58.65 82.9) (layer "F.Cu")
+  (gr_text "Piezo Mic Amplifier v1.0\nDan Larsson 2024" (at 58.65 82.9) (layer "F.Cu")
     (effects (font (size 1.2 1.2) (thickness 0.15)) (justify left bottom))
   )
@@
     (effects (font (size 1 1) (thickness 0.15)) (justify left bottom))
   )
+  (gr_text "WayWayWay" (at 63.948409 54.582682 90) (layer "F.SilkS")
+    (effects (font (size 1 1) (thickness 0.125)) (justify left bottom))
+  )
   (gr_text "+" (at 97.15 70.5) (layer "F.SilkS")
     (effects (font (size 1.5 1.5) (thickness 0.3) bold) (justify left bottom))
   )
-  (gr_text "Piezo Mic Amplifier\nDan Larsson 2024" (at 58.65 82.9) (layer "F.Mask")
+  (gr_text "Piezo Mic Amplifier v1.0\nDan Larsson 2024" (at 58.65 82.9) (layer "F.Mask")
     (effects (font (size 1.2 1.2) (thickness 0.15)) (justify left bottom))
   )
